Commit message: Fix swapped axes in robot model
Between Solidworks and Gazebo, the y and z axes of the coordinate frames
are swapped. This change adapts the robot model to Gazebo's convention
by swapping the y and z axes in the xacros and the STLs.

File: src/kop_description/urdf/kop.xacro (robot description, xacro)
@@ -23,5 +23,5 @@
             <inertial>
                 <origin
-                        xyz="0.3429 -0.039182 -0.4064"
+                        xyz="0.3429 0.4064 -0.039182"
                         rpy="0 0 0"/>
                 <mass value="20.00"/>
@@ -30,7 +30,7 @@
                         ixy="0"
                         ixz="0"
-                        iyy="1.9061"
+                        iyy="0.80739"
                         iyz="0"
-                        izz="0.80739"/>
+                        izz="1.9061"/>
             </inertial>
             <visual>
@@ -46,8 +46,8 @@
             <collision>
                 <origin
-                        xyz="0.3429 -0.039182 -0.4064"
+                        xyz="0.3429 0.4064 -0.039182"
                         rpy="0 0 0"/>
                 <geometry>
-                    <box size="0.6858 0.1188 0.8206"/>
+                    <box size="0.6858 0.8206 0.1188"/>
                 </geometry>
             </collision>

File: src/kop_description/urdf/long_kop.urdf (robot description, URDF)
Before this commit: robot long_kop, 9 links, 8 joints
Links:
- link base_link: geometry collision box size=0.6858 0.8206 0.1188; visual mesh filename=package://kop_description/meshes/visual/small_body.stl
Joints:
- joint hokuyo_joint: origin xyz=0.3429 0.0550 -0.7906 rpy=1.57079632679 1.57079632679 3.14159265359 -> xyz=0.3429 0.7906 0.0550 rpy=0 0 1.57079632679
- joint lf_wheel: origin xyz=0.0657 -0.0563 -0.701 rpy=0 0 0 -> xyz=0.0657 0.701 -0.0563 rpy=0 0 0
- joint lm_wheel: origin xyz=0.0657 -0.0599 -0.4064 rpy=0 0 0 -> xyz=0.0657 0.4064 -0.0599 rpy=0 0 0
- joint lr_wheel: origin xyz=0.0646 -0.0563 -0.1113 rpy=0 0 0 -> xyz=0.0646 0.1113 -0.0563 rpy=0 0 0
- joint rf_wheel: origin xyz=0.6211 -0.0563 -0.7014 rpy=0 0 0 -> xyz=0.6211 0.7014 -0.0563 rpy=0 0 0
- joint rm_wheel: origin xyz=0.6200 -0.0599 -0.4064 rpy=0 0 0 -> xyz=0.6200 0.4064 -0.0599 rpy=0 0 0
- joint rr_wheel: origin xyz=0.6200 -0.0563 -0.1113 rpy=0 0 0 -> xyz=0.6200 0.1113 -0.0563 rpy=0 0 0

File: src/kop_description/urdf/robot.xacro (robot description, xacro)
@@ -10,25 +10,25 @@
             name="left_front"
             short="lf_wheel"
-            origin="0.0657 -0.0563 -0.701"/>
+            origin="0.0657 0.701 -0.0563"/>
     <xacro:insert_wheel
             name="left_middle"
             short="lm_wheel"
-            origin="0.0657 -0.0599 -0.4064"/>
+            origin="0.0657 0.4064 -0.0599"/>
     <xacro:insert_wheel
             name="left_rear"
             short="lr_wheel"
-            origin="0.0646 -0.0563 -0.1113"/>
+            origin="0.0646 0.1113 -0.0563"/>
     <xacro:insert_wheel
             name="right_front"
             short="rf_wheel"
-            origin="0.6211 -0.0563 -0.7014"/>
+            origin="0.6211 0.7014 -0.0563"/>
     <xacro:insert_wheel
             name="right_middle"
             short="rm_wheel"
-            origin="0.6200 -0.0599 -0.4064"/>
+            origin="0.6200 0.4064 -0.0599"/>
     <xacro:insert_wheel
             name="right_rear"
             short="rr_wheel"
-            origin="0.6200 -0.0563 -0.1113"/>
+            origin="0.6200 0.1113 -0.0563"/>
     <xacro:create_trans name="lf_wheel"/>
     <xacro:create_trans name="lm_wheel"/>
@@ -44,5 +44,5 @@
                   min_angle="130"
                   max_angle="-130">
-        <origin xyz="0.3429 0.0550 -0.7906" rpy="${pi / 2.0} ${pi / 2.0} ${pi}"/>
+        <origin xyz="0.3429 0.7906 0.0550" rpy="0 0 ${pi / 2.0}"/>
     </xacro:hokuyo>
     <gazebo>
